File: Zocalo-mcp2551-SOIC.sch (EAGLE design)
At the start: 0 parts

Commit message: fix
Parts:
- added JP1, JP2: (no value), pinhead:PINHD-1X4
- added U1: MCP2551, SparkFun:MCP2551
Connections:
- new net N$1: JP2.4, U1.TXD
- new net N$2: JP2.3, U1.VSS
- new net N$3: JP2.2, U1.VDD
- new net N$4: JP2.1, U1.RXD
- new net N$5: JP1.1, U1.RS
- new net N$6: JP1.2, U1.CANH
- new net N$7: JP1.3, U1.CANL
- new net N$8: JP1.4, U1.VREF
